File: canfd-mc.kicad_pcb (KiCad board)
At the start: 4 copper layers, 55 x 32 mm, 51 parts, among them P1 VBAT, P2 GND, P3 CANH, P4 CANL, U1 ESP32-S3-WROOM-1U-N16R8, U2 MCP2518FDT-E/SL, U3 LM5164DDAR, U4 TCAN332GDR, X1 40MHz 15pF

Commit message: Rev 1.1: 85 C module, through-hole flash header and test pads, 1206 termination
U1 ESP32-S3-WROOM-1U-N8 (the firmware never enables PSRAM). J1 replaces
the seven flat pogo pads with an unfitted 1x7 2.54 mm through-hole header
at the same positions. TP1 (3V3) and TP2 (VIN_PROT) through-hole test
pads on the back. RT1/RT2 as 1206. Silkscreen v1.1. ERC 0, DRC 0,
schematic and board nets match, production files regenerated.

Co-Authored-By: Claude Opus 5 <noreply@anthropic.com>
Parts:
- removed TP3: USB_DP, TestPoint:TestPoint_Pad_D1.5mm
- removed TP4: IO0, TestPoint:TestPoint_Pad_D1.5mm
- removed TP5: ESP_EN, TestPoint:TestPoint_Pad_D1.5mm
- removed TP6: UART_TX, TestPoint:TestPoint_Pad_D1.5mm
- removed TP7: UART_RX, TestPoint:TestPoint_Pad_D1.5mm
- added J1: FLASH, Connector_PinHeader_2.54mm:PinHeader_1x07_P2.54mm_Vertical, B.Cu at (51.5, 55.5)
- RT1, RT2: footprint Resistor_SMD:R_0805_2012Metric -> Resistor_SMD:R_1206_3216Metric
- TP1: value GND -> 3V3; footprint TestPoint:TestPoint_Pad_D1.5mm -> Connector_PinHeader_2.54mm:PinHeader_1x01_P2.54mm_Vertical
- TP2: value USB_DN -> VIN; footprint TestPoint:TestPoint_Pad_D1.5mm -> Connector_PinHeader_2.54mm:PinHeader_1x01_P2.54mm_Vertical
- U1: value ESP32-S3-WROOM-1U-N16R8 -> ESP32-S3-WROOM-1U-N8
- moved TP1 40.3 mm to (88.0, 73.0)
- moved TP2 27.9 mm to (94.0, 62.0)
- moved RT2 0.30 mm to (73.7, 71.4)
Connections:
- TP1 pad 1: GND -> +3V3
- TP2 pad 1: /USB_DN -> /VIN_PROT
Routing:
- net /VIN_PROT: track 21.1 -> 25.5 mm
Other:
- board text added: "CANFD-MC v1.1"
- board text added: "D+"
- board text added: "D-"
- board text added: "EN"
- board text added: "GND"
- board text added: "IO0"
- board text added: "RX"
- board text added: "TX"
- board text removed: "CANFD-MC v1.0 2026-09"
