File: canfd-mc.kicad_sch (KiCad schematic)
At the start: 51 parts, among them P1 VBAT, P2 GND, P3 CANH, P4 CANL, U1 ESP32-S3-WROOM-1U-N16R8, U2 MCP2518FDT-E/SL, U3 LM5164DDAR, U4 TCAN332GDR, X1 40MHz 15pF

Commit message: Rev 1.1: 85 C module, through-hole flash header and test pads, 1206 termination
U1 ESP32-S3-WROOM-1U-N8 (the firmware never enables PSRAM). J1 replaces
the seven flat pogo pads with an unfitted 1x7 2.54 mm through-hole header
at the same positions. TP1 (3V3) and TP2 (VIN_PROT) through-hole test
pads on the back. RT1/RT2 as 1206. Silkscreen v1.1. ERC 0, DRC 0,
schematic and board nets match, production files regenerated.

Co-Authored-By: Claude Opus 5 <noreply@anthropic.com>
Parts:
- removed TP3: USB_DP, TestPoint:TestPoint_Pad_D1.5mm, symbol Connector:TestPoint
- removed TP4: IO0, TestPoint:TestPoint_Pad_D1.5mm, symbol Connector:TestPoint
- removed TP5: ESP_EN, TestPoint:TestPoint_Pad_D1.5mm, symbol Connector:TestPoint
- removed TP6: UART_TX, TestPoint:TestPoint_Pad_D1.5mm, symbol Connector:TestPoint
- removed TP7: UART_RX, TestPoint:TestPoint_Pad_D1.5mm, symbol Connector:TestPoint
- added J1: Flash header 1x7 2.54mm (not fitted), Connector_PinHeader_2.54mm:PinHeader_1x07_P2.54mm_Vertical, symbol Connector_Generic:Conn_01x07
- RT1, RT2: footprint Resistor_SMD:R_0805_2012Metric -> Resistor_SMD:R_1206_3216Metric
- TP1: value GND -> 3V3; footprint TestPoint:TestPoint_Pad_D1.5mm -> Connector_PinHeader_2.54mm:PinHeader_1x01_P2.54mm_Vertical
- TP2: value USB_DN -> VIN; footprint TestPoint:TestPoint_Pad_D1.5mm -> Connector_PinHeader_2.54mm:PinHeader_1x01_P2.54mm_Vertical
- U1: value ESP32-S3-WROOM-1U-N16R8 -> ESP32-S3-WROOM-1U-N8; LCSC C3013946 -> C2980297
Connections:
- net +3V3: now also TP1.1
- net ESP_EN: now also J1.2 (Pin_2)
- net GND: now also J1.1 (Pin_1); no longer TP1.1
- net IO0: now also J1.5 (Pin_5)
- net UART_RX: now also J1.4 (Pin_4)
- net UART_TX: now also J1.3 (Pin_3)
- net USB_DN: now also J1.7 (Pin_7); no longer TP2.1
- net USB_DP: now also J1.6 (Pin_6)
- net VIN_PROT: now also TP2.1
Other:
- note added: "5 Flash header J1 (2.54 mm, not fitted - press-fit a header for the first flash, OTA after that), test pads, power flags"
- note removed: "5 Flash pads (pogo pins, first flash only - OTA after that), power flags"
